File: Channel Display v2.sch (EAGLE design)
At the start: 25 parts, among them IC1 MCP23017SP, IC2 MCP23017SP, IC3 MCP23017SP, IC4 MCP23017SP, IC5 MCP23017SP, IC6 MCP23017SP, IC7 MCP23017SP, IC8 MCP23017SP

Commit message: fixed the header/bus connections, added a 10-pin connector instead of 8 (to handle connection sensing)
Parts:
- H1, H2, SV10, SV11, SV12, SV13, SV14, SV15, SV16, SV3, SV4, SV5, SV6, SV7, SV8, SV9: device con-lstb:MA04-2 -> con-lstb:MA05-2
Connections:
- net +3V3: now also H1.4, H2.4, SV10.4, SV11.4, SV12.4, SV13.4, SV14.4, SV15.4, SV16.4, SV3.4, SV4.4, SV5.4, SV6.4, SV7.4, SV8.4, SV9.4
- net B$2: now also H1.10, H1.9, H2.10, H2.9, SV10.10, SV10.6, SV10.9, SV11.9, SV12.10, SV12.9, SV13.9, SV14.10, SV14.9, SV15.10, SV15.9, SV16.10, SV16.9, SV3.10, SV3.9, SV4.10, SV4.9, SV5.10, SV5.9, SV6.10, SV6.9, SV7.10, SV7.9, SV8.10, SV8.9, SV9.10, SV9.9; no longer H1.4, H2.4, SV10.4, SV11.4, SV12.4, SV13.4, SV14.4, SV15.4, SV16.4, SV3.4, SV4.4, SV5.4, SV6.4, SV7.4, SV8.4, SV9.4
